Commit message: fix: Trunk inertial offset + symmetric *_base_link Y + --no_enable_com_polygon
- t1_simplified.urdf: Trunk inertial origin X gets the -0.0625 compensation
  (was already on visual/collision/spheres per the link comment at L212-216).
  The COM-over-base-polygon cost reads mass-weighted COM via cuRobo's
  state.robot_com; the missing offset shifted Trunk's 11.7 kg contribution
  6.25 cm in +X. Now matches the visible mesh.
- Symmetrize left_base_link Y from 0.08 to 0.084 (right already -0.084).
  After Commit 3 the saved trajectory no longer references *_base_link,
  but internal grasp planning + palm collision spheres are still off
  by 4 mm without this.
- Add TAMPConfiguration.enable_com_polygon and --no_enable_com_polygon
  CLI flag, plumbed through TAMPWorld.get_motion_planner. Previously
  the kwarg existed on get_t1_motion_planner but the call site never
  forwarded it.

S4 (cc.add weight off-by-one) was investigated and REFUTED: cuRobo's
own built-in cost dispatch (cost_manager_robot.py:238, 258, 266, 283)
calls cost_collection.add(value, name) without a weight kwarg in all
four sites, and CostCollection.{clone,merge,copy_at_batch_seed_indices}
all tolerate len(weights) < len(values). Our wrapper at
_curobo_internals.py:264 matches cuRobo's idiom.

Findings: S3, F5, URDF Y-asymm. (S4 refuted.)

Co-Authored-By: Claude Opus 4.7 <noreply@anthropic.com>

File: cutamp/robots/assets/t1_description/t1_simplified.urdf (robot description, URDF)
Before this commit: robot booster_t1_torso, 32 links, 31 joints
Links:
- removed link column_stage_1
- removed link column_stage_2
- removed link column_stage_3
- removed link lifting_base_link
- added link mobile_base_link, mass 20.0; collision box size=0.25 0.25 0.042; visual box size=0.25 0.25 0.042
- added link shank_link, mass 2.0; collision cylinder length=0.28 radius=0.05; visual cylinder length=0.28 radius=0.05
- added link thigh_link, mass 2.0; collision cylinder length=0.236 radius=0.05; visual cylinder length=0.236 radius=0.05
- added link world
Joints:
- removed joint base_to_stage1
- removed joint waist_lift_1
- removed joint waist_lift_2
- added joint ankle_pitch: type revolute, parent mobile_base_link, child shank_link, origin xyz=0 0 0.042 rpy=0 0 0, axis 0 -1 0, limit lower=-0.87 upper=0 effort=12 velocity=18.8
- added joint knee_pitch: type revolute, parent shank_link, child thigh_link, origin xyz=0 0 0.28 rpy=0 0 0, axis 0 -1 0, limit lower=0 upper=2.34 effort=60 velocity=11.7
- added joint world_to_mobile_base: type fixed, parent world, child mobile_base_link, origin xyz=0 0 0 rpy=0 0 0
- joint Left_Elbow_Pitch: limit lower=-2.234 upper=2.234 effort=100 velocity=50 -> lower=-2.234 upper=2.234 effort=100 velocity=18.84
- joint Left_Wrist_Pitch: origin xyz=0 0.105 0.00025 rpy=0 0.19 0 -> xyz=0 0.105 0.00025 rpy=0 0 0
- joint Right_Elbow_Pitch: limit lower=-2.234 upper=2.234 effort=100 velocity=50 -> lower=-2.234 upper=2.234 effort=100 velocity=18.84
- joint Right_Wrist_Pitch: origin xyz=0 -0.105 0.00025 rpy=0 0.19 0 -> xyz=0 -0.105 0.00025 rpy=0 0 0
- joint Torso_Pitch: axis 0 1 0 -> 0 -1 0; limit lower=0 upper=0.7 effort=100 velocity=50 -> lower=-1.8 upper=0 effort=100 velocity=12.5; origin xyz=0 0 0.212388 rpy=0 0 0 -> xyz=0 0 0.236 rpy=0 0 0; parent column_stage_3 -> thigh_link
- joint Waist_Yaw: limit lower=-1.078 upper=1.0198 effort=100 velocity=50 -> lower=-1.57 upper=1.57 effort=30 velocity=10.88
- joint left_base_link: origin xyz=0 0.08 0 rpy=0 0 1.5708 -> xyz=0 0.084 0 rpy=0 0 1.5708
