Commit message: limited torso from pitching backwards.

File: cutamp/robots/assets/t1_description/t1_simplified.urdf (robot description, URDF)
Before this commit: robot booster_t1_torso, 32 links, 31 joints
Joints:
- joint Torso_Pitch: limit lower=-0.7 upper=0.7 effort=100 velocity=50 -> lower=0 upper=0.7 effort=100 velocity=50

Commit message: urdf update

File: cutamp/robots/assets/t1_description/t1_simplified.urdf (robot description, URDF)
Before this commit: robot booster_t1_torso, 32 links, 31 joints
Joints:
- joint AAHead_yaw: limit lower=-1.012 upper=1.012 effort=100 velocity=50 -> lower=-1.02 upper=1.02 effort=7 velocity=12.56
- joint Head_pitch: limit lower=-0.314 upper=0.82 effort=100 velocity=50 -> lower=-0.514 upper=0.85 effort=7 velocity=12.56
- joint Left_Elbow_Pitch: limit lower=-3.14 upper=3.14 effort=100 velocity=50 -> lower=-2.234 upper=2.234 effort=100 velocity=50
- joint Left_Elbow_Yaw: limit lower=-3.14 upper=3.14 effort=100 velocity=50 -> lower=-2.1402 upper=1.6844 effort=18 velocity=18.84
- joint Left_Hand_Roll: limit lower=-3.14 upper=3.14 effort=100 velocity=50 -> lower=-1.3614 upper=1.4285 effort=7 velocity=12.56
- joint Left_Shoulder_Pitch: limit lower=-3.28 upper=1.186 effort=100 velocity=50 -> lower=-3.29 upper=1.18 effort=18 velocity=18.84
- joint Left_Shoulder_Roll: limit lower=-1.64 upper=1.535 effort=100 velocity=50 -> lower=-1.577 upper=1.7055 effort=18 velocity=18.84
- joint Left_Wrist_Pitch: limit lower=-3.14 upper=3.14 effort=100 velocity=50 -> lower=-2.5821 upper=2.5821 effort=7 velocity=12.56; origin xyz=0 0.105 0.00025 rpy=0 0 0 -> xyz=0 0.105 0.00025 rpy=0 0.19 0
- joint Left_Wrist_Yaw: limit lower=-3.14 upper=3.14 effort=100 velocity=50 -> lower=-1.8185 upper=1.4261 effort=18 velocity=18.84
- joint Right_Elbow_Pitch: limit lower=-1.57 upper=1.57 effort=100 velocity=50 -> lower=-2.234 upper=2.234 effort=100 velocity=50
- joint Right_Elbow_Yaw: limit lower=-1.57 upper=1.57 effort=100 velocity=50 -> lower=-1.6844 upper=2.1402 effort=18 velocity=18.84
- joint Right_Hand_Roll: limit lower=-1.57 upper=1.57 effort=100 velocity=50 -> lower=-1.4285 upper=1.3614 effort=7 velocity=12.56
- joint Right_Shoulder_Pitch: limit lower=-1.57 upper=1.57 effort=100 velocity=50 -> lower=-3.29 upper=1.1868 effort=18 velocity=18.84
- joint Right_Shoulder_Roll: limit lower=-1.57 upper=1.57 effort=100 velocity=50 -> lower=-1.7055 upper=1.577 effort=18 velocity=18.84
- joint Right_Wrist_Pitch: limit lower=-1.57 upper=1.57 effort=100 velocity=50 -> lower=-2.5821 upper=2.5821 effort=7 velocity=12.56; origin xyz=0 -0.105 0.00025 rpy=0 0 0 -> xyz=0 -0.105 0.00025 rpy=0 0.19 0
- joint Right_Wrist_Yaw: limit lower=-1.57 upper=1.57 effort=100 velocity=50 -> lower=-1.4261 upper=1.8185 effort=18 velocity=18.84
- joint Waist_Yaw: limit lower=-1.57 upper=1.57 effort=100 velocity=50 -> lower=-1.078 upper=1.0198 effort=100 velocity=50
- joint left_base_link: origin xyz=-0.006 0.08 0.01 rpy=0 0 1.5708 -> xyz=0 0.08 0 rpy=0 0 1.5708
- joint right_base_link: origin xyz=-0.006 -0.084 0.01 rpy=0 0 -1.5708 -> xyz=0 -0.084 0 rpy=0 0 -1.5708

Commit message: adding joint limit margin and tightening joint limits for donwstream mpc

File: cutamp/robots/assets/t1_description/t1_simplified.urdf (robot description, URDF)
Before this commit: robot booster_t1_torso, 32 links, 31 joints
Joints:
- joint Torso_Pitch: limit lower=-1.8 upper=0 effort=100 velocity=12.5 -> lower=-1.7 upper=0 effort=100 velocity=12.5
- joint Waist_Yaw: limit lower=-1.57 upper=1.57 effort=30 velocity=10.88 -> lower=-1.47 upper=1.47 effort=30 velocity=10.88

Commit message: varying heights

File: cutamp/robots/assets/t1_description/t1_simplified.urdf (robot description, URDF)
Before this commit: robot booster_t1_torso, 32 links, 31 joints
Joints:
- joint Torso_Pitch: origin xyz=0 0 0.236 rpy=0 0 0 -> xyz=0.014 0 0.236 rpy=0 0 0
